File: kicad/esp-home-electric-blinds/esp-home-electric-blinds.kicad_pcb (KiCad board)
At the start: 2 copper layers, 56.5 x 99.5 mm, 14 parts, among them J1 AC_IN, J2 Stepper_2_conn, J3 Stepper_2_conn, J4 Conn_01x05, U1 ESP32_mini, U2 TMC2208_Stepper_driver, U3 TMC2208_Stepper_driver

Commit message: power lines
Parts:
- moved F1 44.0 mm to (82.5, 77.5)
- moved U3 36.4 mm to (82.8, 115.4)
- moved U2 12.7 mm to (82.8, 92.4), turned to 180 degrees
- moved U1 0.64 mm to (110.4, 57.7)
Connections:
- net Net-(J1-Pin_1) renamed AC_L
- net Net-(J1-Pin_2) renamed AC_N
Routing:
- net Net-(PS2-+Vout): track 0.00 -> 130.9 mm
- net +3.3V: track 0.00 -> 48.0 mm
- net +12V: track 0.00 -> 27.0 mm
- added copper zone on B.Cu, net AC_L
- added copper zone on F.Cu, net AC_L
- added copper zone on B.Cu, net AC_N
- added copper zone on F.Cu, net AC_N

Commit message: pcb v2
Parts:
- PS1: moved to F.Cu
- moved U3 65.9 mm to (105.1, 53.4)
- moved U1 65.4 mm to (78.0, 114.5), turned to 0 degrees
- moved PS1 45.3 mm to (71.5, 80.0)
- moved U2 39.1 mm to (85.7, 53.4), turned to 0 degrees
- moved J4 16.7 mm to (78.0, 126.2)
- moved H4 12.8 mm to (64.4, 131.0)
- moved J3 10.0 mm to (69.2, 53.4)
- moved H1 9.59 mm to (64.4, 44.0)
- moved H3 8.50 mm to (126.5, 131.0)
- moved J1 8.50 mm to (109.8, 128.8)
- moved PS2 8.50 mm to (110.8, 95.0)
- moved F1 4.46 mm to (86.5, 79.5), turned to 180 degrees
- moved J2 3.74 mm to (121.7, 53.8)
Connections:
- net Net-(PS2-+Vout) renamed DC_VOUT
- J4 pad 5: IO_18 -> GND
- PS1 pad 2: Net-(PS1--VIN) -> GND
- PS2 pad 3: Net-(PS1--VIN) -> GND
Routing:
- net DC_VOUT: track 130.9 -> 0.00 mm
- net +3.3V: track 48.0 -> 135.5 mm
- net EN_PIN: track 0.00 -> 80.7 mm
- net DIR_PIN_2: track 0.00 -> 71.2 mm
- net DIR_PIN: track 0.00 -> 70.4 mm
- net STEP_PIN_2: track 0.00 -> 69.7 mm
- net STEP_PIN: track 0.00 -> 64.5 mm, vias 0 -> 1
- net IO_33: track 0.00 -> 29.3 mm
- net IO_23: track 0.00 -> 24.4 mm
- net IO_32: track 0.00 -> 18.4 mm
- net IO_19: track 0.00 -> 15.7 mm
- net Net-(J3-Pin_2): track 0.00 -> 15.4 mm
- net +12V: track 27.0 -> 41.7 mm
- net Net-(J2-Pin_2): track 0.00 -> 14.6 mm
- net Net-(J3-Pin_1): track 0.00 -> 6.93 mm
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- added copper zone on F.Cu, net +12V
- added copper zone on F.Cu, net DC_VOUT
- added copper zone on B.Cu, net GND
- added copper zone on F.Cu, net GND
- removed copper zone on B.Cu, net AC_L
- removed copper zone on B.Cu, net AC_N
Other:
- board size 56.5 x 99.5 mm -> 66.1 x 91 mm
- board text added: "ESPHome Electric Blinds Author:Jakub Cihanek 26.03.2024 V2.0"
