File: kicad/esp-home-electric-blinds/esp-home-electric-blinds.kicad_sch (KiCad schematic)
At the start: 14 parts, among them J1 AC_IN, J2 Stepper_2_conn, J3 Stepper_2_conn, J4 Conn_01x05, U1 ESP32_mini, U2 TMC2208_Stepper_driver, U3 TMC2208_Stepper_driver

Commit message: pcb v2
Connections:
- net GND: now also J4.5 (Pin_5), PS1.2 (-VIN), PS2.3 (-Vout)
- net IO_18: no longer J4.5 (Pin_5)
- net DC_VOUT: now reaches F1.1, PS2.4 (+Vout)
Changed lines of the file:
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@@
+	)
+	(junction
+		(at 87.63 161.29)
+		(diameter 0)
+		(color 0 0 0 0)
 	)
 	(junction
@@
 	)
 	(junction
+		(at 80.01 156.21)
+		(diameter 0)
+		(color 0 0 0 0)
+	)
+	(junction
+		(at 124.46 163.83)
+		(diameter 0)
+		(color 0 0 0 0)
+	)
+	(junction
 		(at 53.34 161.29)
 		(diameter 0)
@@
 	(wire
 		(pts
-			(xy 77.47 156.21) (xy 83.82 156.21)
+			(xy 77.47 156.21) (xy 80.01 156.21)
 		)
 		(stroke
@@
 	(wire
 		(pts
-			(xy 194.31 237.49) (xy 205.74 237.49)
-		)
-		(stroke
-			(width 0)
-			(type default)
-		)
-	)
-	(wire
-		(pts
 			(xy 53.34 148.59) (xy 53.34 156.21)
 		)
@@
 	(wire
 		(pts
+			(xy 80.01 156.21) (xy 83.82 156.21)
+		)
+		(stroke
+			(width 0)
+			(type default)
+		)
+	)
+	(wire
+		(pts
 			(xy 119.38 156.21) (xy 124.46 156.21)
 		)
@@
 	(wire
 		(pts
-			(xy 124.46 161.29) (xy 124.46 167.64)
+			(xy 124.46 161.29) (xy 124.46 163.83)
 		)
 		(stroke
@@
 	(wire
 		(pts
+			(xy 80.01 146.05) (xy 80.01 156.21)
+		)
+		(stroke
+			(width 0)
+			(type default)
+		)
+	)
+	(wire
+		(pts
 			(xy 355.6 102.87) (xy 347.98 102.87)
 		)
@@
 		)
 	)
+	(wire
+		(pts
+			(xy 87.63 161.29) (xy 87.63 163.83)
+		)
+		(stroke
+			(width 0)
+			(type default)
+		)
+	)
 	(polyline
 		(pts
@@
 	(wire
 		(pts
+			(xy 77.47 146.05) (xy 80.01 146.05)
+		)
+		(stroke
+			(width 0)
+			(type default)
+		)
+	)
+	(wire
+		(pts
 			(xy 353.06 157.48) (xy 353.06 149.86)
 		)
@@
 	(wire
 		(pts
+			(xy 195.58 237.49) (xy 205.74 237.49)
+		)
+		(stroke
+			(width 0)
+			(type default)
+		)
+	)
+	(wire
+		(pts
 			(xy 355.6 177.8) (xy 347.98 177.8)
 		)
@@
 		)
 	)
+	(wire
+		(pts
+			(xy 195.58 240.03) (xy 195.58 237.49)
+		)
+		(stroke
+			(width 0)
+			(type default)
+		)
+	)
+	(wire
+		(pts
+			(xy 87.63 163.83) (xy 124.46 163.83)
+		)
+		(stroke
+			(width 0)
+			(type default)
+		)
+	)
 	(polyline
 		(pts
@@
 	(wire
 		(pts
-			(xy 77.47 161.29) (xy 99.06 161.29)
+			(xy 77.47 161.29) (xy 87.63 161.29)
 		)
 		(stroke
@@
 	(wire
 		(pts
+			(xy 87.63 161.29) (xy 99.06 161.29)
+		)
+		(stroke
+			(width 0)
+			(type default)
+		)
+	)
+	(wire
+		(pts
 			(xy 50.8 148.59) (xy 53.34 148.59)
 		)
@@
 		(pts
 			(xy 236.22 163.83) (xy 236.22 55.88)
+		)
+		(stroke
+			(width 0)
+			(type default)
+		)
+	)
+	(wire
+		(pts
+			(xy 124.46 163.83) (xy 124.46 167.64)
 		)
 		(stroke
@@
 	(global_label "IO_18"
 		(shape input)
-		(at 194.31 237.49 180)
+		(at 209.55 113.03 0)
+		(fields_autoplaced yes)
+		(effects
+			(font
+				(size 1.27 1.27)
+			)
+			(justify left)
+		)
+		(property "Intersheetrefs" "${INTERSHEET_REFS}"
+			(at 217.8571 113.03 0)
+			(effects
+				(font
+					(size 1.27 1.27)
+				)
+				(justify left)
+				(hide yes)
+			)
+		)
+	)
+	(global_label "EN_PIN"
+		(shape input)
+		(at 209.55 107.95 0)
+		(fields_autoplaced yes)
+		(effects
+			(font
+				(size 1.27 1.27)
+			)
+			(justify left)
+		)
+		(property "Intersheetrefs" "${INTERSHEET_REFS}"
+			(at 219.1876 107.95 0)
+			(effects
+				(font
+					(size 1.27 1.27)
+				)
+				(justify left)
+				(hide yes)
+			)
+		)
+	)
+	(global_label "EN_PIN"
+		(shape input)
+		(at 307.34 162.56 180)
 		(fields_autoplaced yes)
 		(effects
@@
 		)
 		(property "Intersheetrefs" "${INTERSHEET_REFS}"
-			(at 186.0029 237.49 0)
+			(at 297.7024 162.56 0)
 			(effects
 				(font
@@
 		)
 	)
-	(global_label "IO_18"
-		(shape input)
-		(at 209.55 113.03 0)
+	(global_label "DIR_PIN"
+		(shape input)
+		(at 309.88 95.25 180)
+		(fields_autoplaced yes)
+		(effects
+			(font
+				(size 1.27 1.27)
+			)
+			(justify right)
+		)
+		(property "Intersheetrefs" "${INTERSHEET_REFS}"
+			(at 299.5771 95.25 0)
+			(effects
+				(font
+					(size 1.27 1.27)
+				)
+				(justify right)
+				(hide yes)
+			)
+		)
+	)
+	(global_label "DIR_PIN"
+		(shape input)
+		(at 208.28 140.97 0)
 		(fields_autoplaced yes)
 		(effects
@@
 		)
 		(property "Intersheetrefs" "${INTERSHEET_REFS}"
-			(at 217.8571 113.03 0)
+			(at 218.5829 140.97 0)
 			(effects
 				(font
@@
 		)
 	)
-	(global_label "EN_PIN"
-		(shape input)
-		(at 209.55 107.95 0)
-		(fields_autoplaced yes)
-		(effects
-			(font
-				(size 1.27 1.27)
-			)
-			(justify left)
-		)
-		(property "Intersheetrefs" "${INTERSHEET_REFS}"
-			(at 219.1876 107.95 0)
-			(effects
-				(font
-					(size 1.27 1.27)
-				)
-				(justify left)
-				(hide yes)
-			)
-		)
-	)
-	(global_label "EN_PIN"
-		(shape input)
-		(at 307.34 162.56 180)
+	(global_label "IO_32"
+		(shape input)
+		(at 203.2 229.87 180)
 		(fields_autoplaced yes)
 		(effects
@@
 		)
 		(property "Intersheetrefs" "${INTERSHEET_REFS}"
-			(at 297.7024 162.56 0)
+			(at 194.8929 229.87 0)
 			(effects
 				(font
@@
 		)
 	)
-	(global_label "DIR_PIN"
-		(shape input)
-		(at 309.88 95.25 180)
+	(global_label "DC_VOUT"
+		(shape input)
+		(at 77.47 146.05 180)
 		(fields_autoplaced yes)
 		(effects
@@
 		)
 		(property "Intersheetrefs" "${INTERSHEET_REFS}"
-			(at 299.5771 95.25 0)
-			(effects
-				(font
-					(size 1.27 1.27)
-				)
-				(justify right)
-				(hide yes)
-			)
-		)
-	)
-	(global_label "DIR_PIN"
-		(shape input)
-		(at 208.28 140.97 0)
-		(fields_autoplaced yes)
-		(effects
-			(font
-				(size 1.27 1.27)
-			)
-			(justify left)
-		)
-		(property "Intersheetrefs" "${INTERSHEET_REFS}"
-			(at 218.5829 140.97 0)
-			(effects
-				(font
-					(size 1.27 1.27)
-				)
-				(justify left)
-				(hide yes)
-			)
-		)
-	)
-	(global_label "IO_32"
-		(shape input)
-		(at 203.2 229.87 180)
-		(fields_autoplaced yes)
-		(effects
-			(font
-				(size 1.27 1.27)
-			)
-			(justify right)
-		)
-		(property "Intersheetrefs" "${INTERSHEET_REFS}"
-			(at 194.8929 229.87 0)
+			(at 66.26 146.05 0)
 			(effects
 				(font
@@
 					(unit 1)
 				)
+			)
+		)
+	)
+	(symbol
+		(lib_id "power:GND")
+		(at 195.58 240.03 0)
+		(unit 1)
+		(exclude_from_sim no)
+		(in_bom yes)
+		(on_board yes)
+		(dnp no)
+		(fields_autoplaced yes)
+		(property "Reference" "#PWR012"
+			(at 195.58 246.38 0)
+			(effects
+				(font
+					(size 1.27 1.27)
+				)
+				(hide yes)
+			)
+		)
+		(property "Value" "GND"
+			(at 195.58 245.11 0)
+			(effects
+				(font
+					(size 1.27 1.27)
+				)
+			)
+		)
+		(property "Footprint" ""
+			(at 195.58 240.03 0)
+			(effects
+				(font
+					(size 1.27 1.27)
+				)
+				(hide yes)
+			)
+		)
+		(property "Datasheet" ""
+			(at 195.58 240.03 0)
+			(effects
+				(font
+					(size 1.27 1.27)
+				)
+				(hide yes)
+			)
+		)
+		(property "Description" "Power symbol creates a global label with name \"GND\" , ground"
+			(at 195.58 240.03 0)
+			(effects
+				(font
+					(size 1.27 1.27)
+				)
+				(hide yes)
+			)
+		)
+		(pin "1"
+		)
+		(instances
+			(project "esp-home-electric-blinds"
+				(path "/07d3a4e0-56e5-4d89-afd4-c6828a783612"
+					(reference "#PWR012")
+					(unit 1)
+				)

Commit message: added stepper connector
Parts:
- added J5: Stepper_2_conn, connectors_johnymalina:JST_smd_1x04_horizontal, symbol Connector_Generic:Conn_01x04
- added J6: Stepper_1_conn, connectors_johnymalina:JST_smd_1x04_horizontal, symbol Connector_Generic:Conn_01x04
- J3: value Stepper_2_conn -> Stepper_1_conn
Connections:
- net at J3.1 (Pin_1), U2.JP2_4 (OA1): now also J6.1 (Pin_1)
- net at J3.2 (Pin_2), U2.JP2_3 (OA2): now also J6.2 (Pin_2)
- net at J3.3 (Pin_3), U2.JP2_5 (OB1): now also J6.3 (Pin_3)
- net at J3.4 (Pin_4), U2.JP2_6 (OB2): now also J6.4 (Pin_4)
- net at J2.1 (Pin_1), U3.JP2_4 (OA1): now also J5.1 (Pin_1)
- net at J2.2 (Pin_2), U3.JP2_3 (OA2): now also J5.2 (Pin_2)
- net at J2.3 (Pin_3), U3.JP2_5 (OB1): now also J5.3 (Pin_3)
- net at J2.4 (Pin_4), U3.JP2_6 (OB2): now also J5.4 (Pin_4)
Other:
- moved on the sheet: J2, J3

Commit message: stepper pinout switch
Connections:
- net at J3.3 (Pin_3), J6.3 (Pin_3): now also U2.JP2_6 (OB2); no longer U2.JP2_5 (OB1)
- net at J3.4 (Pin_4), J6.4 (Pin_4): now also U2.JP2_5 (OB1); no longer U2.JP2_6 (OB2)
- net at J2.3 (Pin_3), J5.3 (Pin_3): now also U3.JP2_6 (OB2); no longer U3.JP2_5 (OB1)
- net at J2.4 (Pin_4), J5.4 (Pin_4): now also U3.JP2_5 (OB1); no longer U3.JP2_6 (OB2)
Changed lines of the file:
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@@
+	)
+	(junction
+		(at 356.87 172.72)
+		(diameter 0)
+		(color 0 0 0 0)
+	)
+	(junction
+		(at 354.33 110.49)
+		(diameter 0)
+		(color 0 0 0 0)
 	)
 	(junction
@@
 	)
 	(junction
-		(at 356.87 172.72)
+		(at 359.41 100.33)
+		(diameter 0)
+		(color 0 0 0 0)
+	)
+	(junction
+		(at 361.95 97.79)
+		(diameter 0)
+		(color 0 0 0 0)
+	)
+	(junction
+		(at 87.63 161.29)
+		(diameter 0)
+		(color 0 0 0 0)
+	)
+	(junction
+		(at 351.79 180.34)
+		(diameter 0)
+		(color 0 0 0 0)
+	)
+	(junction
+		(at 95.25 156.21)
+		(diameter 0)
+		(color 0 0 0 0)
+	)
+	(junction
+		(at 80.01 156.21)
+		(diameter 0)
+		(color 0 0 0 0)
+	)
+	(junction
+		(at 124.46 163.83)
 		(diameter 0)
 		(color 0 0 0 0)
@@
 	)
 	(junction
-		(at 351.79 177.8)
-		(diameter 0)
-		(color 0 0 0 0)
-	)
-	(junction
-		(at 354.33 105.41)
-		(diameter 0)
-		(color 0 0 0 0)
-	)
-	(junction
-		(at 359.41 100.33)
-		(diameter 0)
-		(color 0 0 0 0)
-	)
-	(junction
-		(at 361.95 97.79)
-		(diameter 0)
-		(color 0 0 0 0)
-	)
-	(junction
-		(at 87.63 161.29)
-		(diameter 0)
-		(color 0 0 0 0)
-	)
-	(junction
-		(at 95.25 156.21)
-		(diameter 0)
-		(color 0 0 0 0)
-	)
-	(junction
-		(at 80.01 156.21)
-		(diameter 0)
-		(color 0 0 0 0)
-	)
-	(junction
-		(at 124.46 163.83)
-		(diameter 0)
-		(color 0 0 0 0)
-	)
-	(junction
 		(at 53.34 161.29)
 		(diameter 0)
@@
 	(wire
 		(pts
+			(xy 351.79 105.41) (xy 351.79 102.87)
+		)
+		(stroke
+			(width 0)
+			(type default)
+		)
+	)
+	(wire
+		(pts
 			(xy 209.55 90.17) (xy 205.74 90.17)
 		)
@@
 	(wire
 		(pts
+			(xy 349.25 175.26) (xy 349.25 180.34)
+		)
+		(stroke
+			(width 0)
+			(type default)
+		)
+	)
+	(wire
+		(pts
 			(xy 48.26 157.48) (xy 53.34 157.48)
 		)
@@
 		)
 	)
+	(wire
+		(pts
+			(xy 350.52 177.8) (xy 350.52 175.26)
+		)
+		(stroke
+			(width 0)
+			(type default)
+		)
+	)
 	(polyline
 		(pts
@@
 	(wire
 		(pts
+			(xy 347.98 177.8) (xy 350.52 177.8)
+		)
+		(stroke
+			(width 0)
+			(type default)
+		)
+	)
+	(wire
+		(pts
 			(xy 53.34 148.59) (xy 53.34 156.21)
 		)
@@
 	(wire
 		(pts
-			(xy 354.33 105.41) (xy 347.98 105.41)
-		)
-		(stroke
-			(width 0)
-			(type default)
-		)
-	)
-	(wire
-		(pts
 			(xy 179.07 74.93) (xy 179.07 80.01)
 		)
@@
 	(wire
 		(pts
+			(xy 347.98 105.41) (xy 351.79 105.41)
+		)
+		(stroke
+			(width 0)
+			(type default)
+		)
+	)
+	(wire
+		(pts
 			(xy 219.71 115.57) (xy 205.74 115.57)
 		)
@@
 	(wire
 		(pts
+			(xy 350.52 175.26) (xy 354.33 175.26)
+		)
+		(stroke
+			(width 0)
+			(type default)
+		)
+	)
+	(wire
+		(pts
 			(xy 219.71 120.65) (xy 205.74 120.65)
 		)
@@
 		)
 	)
+	(wire
+		(pts
+			(xy 349.25 180.34) (xy 351.79 180.34)
+		)
+		(stroke
+			(width 0)
+			(type default)
+		)
+	)
 	(polyline
 		(pts
@@
 	(wire
 		(pts
-			(xy 356.87 102.87) (xy 347.98 102.87)
+			(xy 347.98 102.87) (xy 350.52 102.87)
 		)
 		(stroke
@@
 	(wire
 		(pts
+			(xy 351.79 102.87) (xy 356.87 102.87)
+		)
+		(stroke
+			(width 0)
+			(type default)
+		)
+	)
+	(wire
+		(pts
 			(xy 359.41 100.33) (xy 347.98 100.33)
 		)
@@
 	(wire
 		(pts
-			(xy 354.33 116.84) (xy 354.33 105.41)
-		)
-		(stroke
-			(width 0)
-			(type default)
-		)
-	)
-	(wire
-		(pts
-			(xy 354.33 175.26) (xy 347.98 175.26)
+			(xy 354.33 116.84) (xy 354.33 110.49)
 		)
 		(stroke
@@
 	(wire
 		(pts
+			(xy 350.52 110.49) (xy 354.33 110.49)
+		)
+		(stroke
+			(width 0)
+			(type default)
+		)
+	)
+	(wire
+		(pts
 			(xy 367.03 97.79) (xy 361.95 97.79)
 		)
@@
 	(wire
 		(pts
-			(xy 351.79 177.8) (xy 347.98 177.8)
+			(xy 347.98 175.26) (xy 349.25 175.26)
 		)
 		(stroke
@@
 	(wire
 		(pts
+			(xy 354.33 110.49) (xy 354.33 105.41)
+		)
+		(stroke
+			(width 0)
+			(type default)
+		)
+	)
+	(wire
+		(pts
 			(xy 50.8 148.59) (xy 53.34 148.59)
 		)
@@
 	(wire
 		(pts
+			(xy 351.79 180.34) (xy 351.79 177.8)
+		)
+		(stroke
+			(width 0)
+			(type default)
+		)
+	)
+	(wire
+		(pts
 			(xy 364.49 186.69) (xy 354.33 186.69)
 		)
@@
 	(wire
 		(pts
-			(xy 351.79 189.23) (xy 351.79 177.8)
+			(xy 351.79 189.23) (xy 351.79 180.34)
 		)
 		(stroke
@@
 		)
 		(stroke
+			(width 0)
+			(type default)
+		)
+	)
+	(wire
+		(pts
+			(xy 350.52 102.87) (xy 350.52 110.49)
+		)
+		(stroke

Commit message: stepper connection update
Connections:
- net at J3.1 (Pin_1), J6.1 (Pin_1): now also U2.JP2_6 (OB2); no longer U2.JP2_4 (OA1)
- net at J3.2 (Pin_2), J6.2 (Pin_2): now also U2.JP2_5 (OB1); no longer U2.JP2_3 (OA2)
- net at J3.3 (Pin_3), J6.3 (Pin_3): now also U2.JP2_4 (OA1); no longer U2.JP2_6 (OB2)
- net at J3.4 (Pin_4), J6.4 (Pin_4): now also U2.JP2_3 (OA2); no longer U2.JP2_5 (OB1)
- net at J2.1 (Pin_1), J5.1 (Pin_1): now also U3.JP2_6 (OB2); no longer U3.JP2_4 (OA1)
- net at J2.2 (Pin_2), J5.2 (Pin_2): now also U3.JP2_5 (OB1); no longer U3.JP2_3 (OA2)
- net at J2.3 (Pin_3), J5.3 (Pin_3): now also U3.JP2_4 (OA1); no longer U3.JP2_6 (OB2)
- net at J2.4 (Pin_4), J5.4 (Pin_4): now also U3.JP2_3 (OA2); no longer U3.JP2_5 (OB1)
Other:
- moved on the sheet: J2, J3, J5, J6

Commit message: pcb V2
Connections:
- net +3.3V: now also J4.4 (Pin_4)
- net EN_PIN: no longer U3.JP1_8 (EN)
- net IO_19: now also J4.2 (Pin_2); no longer J4.4 (Pin_4)
- net IO_32 renamed EN_PIN_2
- net EN_PIN_2: now also U3.JP1_8 (EN); no longer J4.2 (Pin_2)
